File: ESP12 Altherma.brd (EAGLE design)
At the start: 80.1 x 49.8 mm, 51 parts, among them J1 Thermo Rly, J2 X85A - PL, K1 HRS1KH-S_DC5V, K2 HRS1KH-S_DC5V, P1 X10A, U1 TLP291-4(GB-TP,E), U2 AP2112K-3.3TRG1, U4 DRDC3105E6-7, U5 SN74LVC1G125GV

Commit message: I think this is v1.0. This commit free of any panelisation guff.
Parts:
- removed SG: (no value), SparkFun-Connectors:1X04_LOCK
- removed SJ3: SOLDERJUMPERTRACE, Master 2016:SJ_2S-TRACE
- added CONN4: SG, SparkFun-Connectors:1X04
- added LED5: (no value), Master 2016:LED-1206
- added R17: 180R, Master 2016:1206
- added SJ1: SOLDERJUMPERTRACE, Master 2016:SJ_2S-TRACE
- U1: value TLP291-4(GB-TP,E) -> TLP291-4
- U2: value AP2112K-3.3TRG1 -> AP2112K-3.3
- moved D2 0.63 mm to (64.8, 36.2)
- moved S1 0.63 mm to (58.4, 43.8)
- moved S2 0.63 mm to (66.7, 43.8)
- renumbered J1 to CON5, J2 to CON2, P1 to CON3, R19 to R16, SV1 to CON1
Connections:
- new net N$28: LED5.C, R17.2
- net GPIO2: now also R17.1
- net N$14: now also SJ1.1; no longer SJ3.1
- net N$22: now also CONN4.1; no longer SG.1
- net N$23: now also CONN4.2; no longer SG.2
- net N$24: now also CONN4.3; no longer SG.3
- net N$25: now also CONN4.4; no longer SG.4
- net N$5: now also SJ1.2; no longer SJ3.2
- net VCC: now also LED5.A
Routing:
- net VCC: track 127.6 -> 144.2 mm
- net GPIO2: track 7.04 -> 15.3 mm, vias 0 -> 1
- net GPIO0: track 68.8 -> 63.5 mm
- net RXD: track 65.4 -> 60.1 mm
- net N$28: track 0.00 -> 3.58 mm
- net TXD: track 66.0 -> 62.6 mm
- net N$22: track 22.0 -> 19.9 mm
- net GND: track 22.6 -> 21.8 mm
- net N$5: track 3.38 -> 2.67 mm
- net RST: track 28.0 -> 28.6 mm
Other:
- board text added: "1"
- board text added: "5V"
- board text added: "G"
- board text added: "OK"
- board text added: "SG1"
- board text added: "SG2"
- board text added: "Sig"
- board text added: "Smart Gd"
- board text removed: "AP2112"
- board text removed: "C1"
- board text removed: "C2"
- board text removed: "C3"
- board text removed: "D1"
- board text removed: "D2"
- board text removed: "EP1"
- board text removed: "EP2"
- board text removed: "JP1"
- board text removed: "JP2"
- board text removed: "JP3"
- board text removed: "JP4"
- board text removed: "JP5"
- board text removed: "JP6"
- board text removed: "JP7"
- board text removed: "JP8"
- board text removed: "JP9"
- board text removed: "LED1"
- board text removed: "LED2"
- board text removed: "Q1"
- board text removed: "R1"
- board text removed: "R10"
- board text removed: "R11"
- board text removed: "R12"
- board text removed: "R2"
- board text removed: "R3"
- board text removed: "R4"
- board text removed: "R5"
- board text removed: "R6"
- board text removed: "R7"
- board text removed: "R8"
- board text removed: "R9"
- board text removed: "S1"
- board text removed: "S2"
- board text removed: "SJ1"
- board text removed: "SJ2"
- board text removed: "SJ3"
- board text removed: "SJR1"
- board text removed: "U$1"
- board text removed: "U2"
