File: ESP12 Altherma.sch (EAGLE design)
At the start: 58 parts, among them J1 455-1750-1-ND, K1 HRS1KH-S_DC5V, K2 HRS1KH-S_DC5V, U1 TLP291-4(GB-TP,E), U2 AP2112K-3.3TRG1, U4 DRDC3105E6-7, U5 SN74LVC1G125GV

Commit message: shorten board. share GPIO for LP and SG. use JST connectors. tidy needless complexity
Parts:
- removed EP1: Ext Pwr, con-amp-quick:M02S
- removed EP3: (no value), Master 2016:USB-FCI_SMD***
- removed LED5, LED6, LED7: (no value), Master 2016:LED1206
- removed R16, R17, R18: 180R, Master 2016:R-EU_
- removed SJ1: 3V3 | 5V, Master 2016:SOLDERJUMPER_2WAYSJ_3_TRACE
- removed X10: (no value), SparkFun-Connectors:CONN_05
- removed X85A: (no value), SparkFun-Connectors:CONN_06FEMALE_LOCK
- added J2: X85A - PL, conn-jst-pa6:B06B-PASK(LF)(SN)
- added JP4: PL En, SparkFun-Passives:JUMPER-2PTH
- added P1: X10A, con-jst-eh:B5B-EH-A
- JP2: value Pwr by Serial -> Pwr Serial
- S2: value Flash/Cmd -> Flash
- SV1: value Serial -> PGM/BT Serial
Connections:
- removed net N$28: J1.3, SJ1.2
- removed net N$30: LED6.C, R17.2
- removed net N$31: LED7.C, R18.2
- net 5V: now also J1.3, U5.VCC; no longer EP1-1.S, EP3.VBUS, SJ1.3
- net 5V_HP: now also P1.1; no longer U5.VCC, X10.1
- net GND: now also P1.5; no longer EP1-2.S, EP3.GND, X10.5
- net GPIO0: no longer LED1.A, R9.2
- net GPIO14: now also LED2.A, R8.2; no longer LED5.A
- net GPIO16: now also LED1.A, R9.2; no longer LED6.A
- net GPIO2: no longer LED2.A, R8.2
- net GPIO5: no longer LED7.A
- net N$11: now also J2.5; no longer X85A.5
- net N$12: now also J2.4; no longer X85A.4
- net N$13: now also J2.2; no longer X85A.2
- net N$20: now also P1.3; no longer X10.3
- net N$21: now also P1.2; no longer X10.2
- net N$27: now also J2.6, JP4.1; no longer LED5.C, R16.2
- net N$3: now also J2.3; no longer X85A.3
- net N$4: no longer R16.1, R17.1, R18.1
- net VCC: no longer SJ1.1
- net X85_GND: now also JP4.2; no longer X85A.6
Other:
- note added: "Move?"
- moved on the sheet: JP1, LED1, LED2, LED3, LED4, R12, R13, R14, R15

Commit message: change esp12 to version without Restrict layer so I can panelise
Parts:
- SJR1: device esp12e:ESP8266-12EESP12E -> esp12e:ESP8266-12EESP8266-ESP12E-X
Changed lines of the file:
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@@
 <grid distance="0.1" unitdist="inch" unit="inch" style="lines" multiple="1" display="yes" altdistance="0.05" altunitdist="inch" altunit="inch"/>
 <layers>
-<layer number="1" name="Top" color="4" fill="1" visible="no" active="no"/>
-<layer number="16" name="Bottom" color="1" fill="1" visible="no" active="no"/>
-<layer number="17" name="Pads" color="2" fill="1" visible="no" active="no"/>
-<layer number="18" name="Vias" color="2" fill="1" visible="no" active="no"/>
-<layer number="19" name="Unrouted" color="6" fill="1" visible="no" active="no"/>
-<layer number="20" name="Dimension" color="15" fill="1" visible="no" active="no"/>
-<layer number="21" name="tPlace" color="16" fill="1" visible="no" active="no"/>
-<layer number="22" name="bPlace" color="14" fill="1" visible="no" active="no"/>
-<layer number="23" name="tOrigins" color="15" fill="1" visible="no" active="no"/>
-<layer number="24" name="bOrigins" color="15" fill="1" visible="no" active="no"/>
-<layer number="25" name="tNames" color="7" fill="1" visible="no" active="no"/>
-<layer number="26" name="bNames" color="7" fill="1" visible="no" active="no"/>
-<layer number="27" name="tValues" color="24" fill="1" visible="no" active="no"/>
-<layer number="28" name="bValues" color="24" fill="1" visible="no" active="no"/>
+<layer number="1" name="Top" color="4" fill="1" visible="yes" active="no"/>
+<layer number="16" name="Bottom" color="1" fill="1" visible="yes" active="no"/>
+<layer number="17" name="Pads" color="2" fill="1" visible="yes" active="no"/>
+<layer number="18" name="Vias" color="2" fill="1" visible="yes" active="no"/>
+<layer number="19" name="Unrouted" color="6" fill="1" visible="yes" active="no"/>
+<layer number="20" name="Dimension" color="15" fill="1" visible="yes" active="no"/>
+<layer number="21" name="tPlace" color="16" fill="1" visible="yes" active="no"/>
+<layer number="22" name="bPlace" color="14" fill="1" visible="yes" active="no"/>
+<layer number="23" name="tOrigins" color="15" fill="1" visible="yes" active="no"/>
+<layer number="24" name="bOrigins" color="15" fill="1" visible="yes" active="no"/>
+<layer number="25" name="tNames" color="7" fill="1" visible="yes" active="no"/>
+<layer number="26" name="bNames" color="7" fill="1" visible="yes" active="no"/>
+<layer number="27" name="tValues" color="24" fill="1" visible="yes" active="no"/>
+<layer number="28" name="bValues" color="24" fill="1" visible="yes" active="no"/>
 <layer number="29" name="tStop" color="7" fill="3" visible="no" active="no"/>
 <layer number="30" name="bStop" color="7" fill="6" visible="no" active="no"/>
@@
 <layer number="35" name="tGlue" color="7" fill="4" visible="no" active="no"/>
 <layer number="36" name="bGlue" color="7" fill="5" visible="no" active="no"/>
-<layer number="37" name="tTest" color="7" fill="1" visible="no" active="no"/>
-<layer number="38" name="bTest" color="7" fill="1" visible="no" active="no"/>
+<layer number="37" name="tTest" color="7" fill="1" visible="yes" active="no"/>
+<layer number="38" name="bTest" color="7" fill="1" visible="yes" active="no"/>
 <layer number="39" name="tKeepout" color="4" fill="11" visible="no" active="no"/>
 <layer number="40" name="bKeepout" color="1" fill="11" visible="no" active="no"/>
@@
 <layer number="44" name="Drills" color="7" fill="1" visible="no" active="no"/>
 <layer number="45" name="Holes" color="7" fill="1" visible="no" active="no"/>
-<layer number="46" name="Milling" color="3" fill="1" visible="no" active="no"/>
-<layer number="47" name="Measures" color="7" fill="1" visible="no" active="no"/>
-<layer number="48" name="Document" color="7" fill="1" visible="no" active="no"/>
-<layer number="49" name="Reference" color="7" fill="1" visible="no" active="no"/>
-<layer number="50" name="dxf" color="7" fill="1" visible="no" active="no"/>
-<layer number="51" name="tDocu" color="6" fill="1" visible="no" active="no"/>
-<layer number="52" name="bDocu" color="7" fill="1" visible="no" active="no"/>
-<layer number="53" name="tGND_GNDA" color="7" fill="9" visible="no" active="no"/>
-<layer number="54" name="bGND_GNDA" color="1" fill="9" visible="no" active="no"/>
-<layer number="56" name="wert" color="7" fill="1" visible="no" active="no"/>
-<layer number="57" name="tCAD" color="7" fill="1" visible="no" active="no"/>
-<layer number="58" name="bCAD" color="7" fill="1" visible="no" active="no"/>
-<layer number="59" name="tCarbon" color="7" fill="1" visible="no" active="no"/>
-<layer number="60" name="bCarbon" color="7" fill="1" visible="no" active="no"/>
+<layer number="46" name="Milling" color="3" fill="1" visible="yes" active="no"/>
+<layer number="47" name="Measures" color="7" fill="1" visible="yes" active="no"/>
+<layer number="48" name="Document" color="7" fill="1" visible="yes" active="no"/>
+<layer number="49" name="Reference" color="7" fill="1" visible="yes" active="no"/>
+<layer number="50" name="dxf" color="7" fill="1" visible="yes" active="no"/>
+<layer number="51" name="tDocu" color="6" fill="1" visible="yes" active="no"/>
+<layer number="52" name="bDocu" color="7" fill="1" visible="yes" active="no"/>
+<layer number="53" name="tGND_GNDA" color="7" fill="9" visible="yes" active="no"/>
+<layer number="54" name="bGND_GNDA" color="1" fill="9" visible="yes" active="no"/>
+<layer number="56" name="wert" color="7" fill="1" visible="yes" active="no"/>
+<layer number="57" name="tCAD" color="7" fill="1" visible="yes" active="no"/>
+<layer number="58" name="bCAD" color="7" fill="1" visible="yes" active="no"/>
+<layer number="59" name="tCarbon" color="7" fill="1" visible="yes" active="no"/>
+<layer number="60" name="bCarbon" color="7" fill="1" visible="yes" active="no"/>
 <layer number="88" name="SimResults" color="9" fill="1" visible="yes" active="yes"/>
 <layer number="89" name="SimProbes" color="9" fill="1" visible="yes" active="yes"/>
@@
 </classes>
 <parts>
-<part name="SJR1" library="esp12e" deviceset="ESP8266-12E" device="ESP12E"/>
+<part name="SJR1" library="esp12e" deviceset="ESP8266-12E" device="ESP8266-ESP12E-X"/>
 <part name="GND1" library="Master" deviceset="GND" device=""/>
 <part name="GND2" library="Master" deviceset="GND" device=""/>

Commit message: Provisionally final tweaks prior to attempting panelisation
Parts:
- added JP5: SG En, SparkFun-Passives:JUMPER-2PTH
- J1: value 455-1750-1-ND -> Thermo Rly
- JP3: value Signals -> LED En
Connections:
- new net N$6: JP5.1, K1.2, K2.2
- net 5V: now also JP5.2; no longer K1.2, K2.2
Changed lines of the file:
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@@
 <grid distance="0.1" unitdist="inch" unit="inch" style="lines" multiple="1" display="yes" altdistance="0.05" altunitdist="inch" altunit="inch"/>
 <layers>
-<layer number="1" name="Top" color="4" fill="1" visible="yes" active="no"/>
-<layer number="16" name="Bottom" color="1" fill="1" visible="yes" active="no"/>
-<layer number="17" name="Pads" color="2" fill="1" visible="yes" active="no"/>
-<layer number="18" name="Vias" color="2" fill="1" visible="yes" active="no"/>
-<layer number="19" name="Unrouted" color="6" fill="1" visible="yes" active="no"/>
-<layer number="20" name="Dimension" color="15" fill="1" visible="yes" active="no"/>
-<layer number="21" name="tPlace" color="16" fill="1" visible="yes" active="no"/>
-<layer number="22" name="bPlace" color="14" fill="1" visible="yes" active="no"/>
-<layer number="23" name="tOrigins" color="15" fill="1" visible="yes" active="no"/>
-<layer number="24" name="bOrigins" color="15" fill="1" visible="yes" active="no"/>
-<layer number="25" name="tNames" color="7" fill="1" visible="yes" active="no"/>
-<layer number="26" name="bNames" color="7" fill="1" visible="yes" active="no"/>
-<layer number="27" name="tValues" color="24" fill="1" visible="yes" active="no"/>
-<layer number="28" name="bValues" color="24" fill="1" visible="yes" active="no"/>
+<layer number="1" name="Top" color="4" fill="1" visible="no" active="no"/>
+<layer number="16" name="Bottom" color="1" fill="1" visible="no" active="no"/>
+<layer number="17" name="Pads" color="2" fill="1" visible="no" active="no"/>
+<layer number="18" name="Vias" color="2" fill="1" visible="no" active="no"/>
+<layer number="19" name="Unrouted" color="6" fill="1" visible="no" active="no"/>
+<layer number="20" name="Dimension" color="15" fill="1" visible="no" active="no"/>
+<layer number="21" name="tPlace" color="16" fill="1" visible="no" active="no"/>
+<layer number="22" name="bPlace" color="14" fill="1" visible="no" active="no"/>
+<layer number="23" name="tOrigins" color="15" fill="1" visible="no" active="no"/>
+<layer number="24" name="bOrigins" color="15" fill="1" visible="no" active="no"/>
+<layer number="25" name="tNames" color="7" fill="1" visible="no" active="no"/>
+<layer number="26" name="bNames" color="7" fill="1" visible="no" active="no"/>
+<layer number="27" name="tValues" color="24" fill="1" visible="no" active="no"/>
+<layer number="28" name="bValues" color="24" fill="1" visible="no" active="no"/>
 <layer number="29" name="tStop" color="7" fill="3" visible="no" active="no"/>
 <layer number="30" name="bStop" color="7" fill="6" visible="no" active="no"/>
@@
 <layer number="35" name="tGlue" color="7" fill="4" visible="no" active="no"/>
 <layer number="36" name="bGlue" color="7" fill="5" visible="no" active="no"/>
-<layer number="37" name="tTest" color="7" fill="1" visible="yes" active="no"/>
-<layer number="38" name="bTest" color="7" fill="1" visible="yes" active="no"/>
+<layer number="37" name="tTest" color="7" fill="1" visible="no" active="no"/>
+<layer number="38" name="bTest" color="7" fill="1" visible="no" active="no"/>
 <layer number="39" name="tKeepout" color="4" fill="11" visible="no" active="no"/>
 <layer number="40" name="bKeepout" color="1" fill="11" visible="no" active="no"/>
@@
 <layer number="44" name="Drills" color="7" fill="1" visible="no" active="no"/>
 <layer number="45" name="Holes" color="7" fill="1" visible="no" active="no"/>
-<layer number="46" name="Milling" color="3" fill="1" visible="yes" active="no"/>
-<layer number="47" name="Measures" color="7" fill="1" visible="yes" active="no"/>
-<layer number="48" name="Document" color="7" fill="1" visible="yes" active="no"/>
-<layer number="49" name="Reference" color="7" fill="1" visible="yes" active="no"/>
-<layer number="50" name="dxf" color="7" fill="1" visible="yes" active="no"/>
-<layer number="51" name="tDocu" color="6" fill="1" visible="yes" active="no"/>
-<layer number="52" name="bDocu" color="7" fill="1" visible="yes" active="no"/>
-<layer number="53" name="tGND_GNDA" color="7" fill="9" visible="yes" active="no"/>
-<layer number="54" name="bGND_GNDA" color="1" fill="9" visible="yes" active="no"/>
-<layer number="56" name="wert" color="7" fill="1" visible="yes" active="no"/>
-<layer number="57" name="tCAD" color="7" fill="1" visible="yes" active="no"/>
-<layer number="58" name="bCAD" color="7" fill="1" visible="yes" active="no"/>
-<layer number="59" name="tCarbon" color="7" fill="1" visible="yes" active="no"/>
-<layer number="60" name="bCarbon" color="7" fill="1" visible="yes" active="no"/>
+<layer number="46" name="Milling" color="3" fill="1" visible="no" active="no"/>
+<layer number="47" name="Measures" color="7" fill="1" visible="no" active="no"/>
+<layer number="48" name="Document" color="7" fill="1" visible="no" active="no"/>
+<layer number="49" name="Reference" color="7" fill="1" visible="no" active="no"/>
+<layer number="50" name="dxf" color="7" fill="1" visible="no" active="no"/>
+<layer number="51" name="tDocu" color="6" fill="1" visible="no" active="no"/>
+<layer number="52" name="bDocu" color="7" fill="1" visible="no" active="no"/>
+<layer number="53" name="tGND_GNDA" color="7" fill="9" visible="no" active="no"/>
+<layer number="54" name="bGND_GNDA" color="1" fill="9" visible="no" active="no"/>
+<layer number="56" name="wert" color="7" fill="1" visible="no" active="no"/>
+<layer number="57" name="tCAD" color="7" fill="1" visible="no" active="no"/>
+<layer number="58" name="bCAD" color="7" fill="1" visible="no" active="no"/>
+<layer number="59" name="tCarbon" color="7" fill="1" visible="no" active="no"/>
+<layer number="60" name="bCarbon" color="7" fill="1" visible="no" active="no"/>
 <layer number="88" name="SimResults" color="9" fill="1" visible="yes" active="yes"/>
 <layer number="89" name="SimProbes" color="9" fill="1" visible="yes" active="yes"/>
@@
 <part name="LED2" library="Master 2016" deviceset="LED" device="1206"/>
 <part name="LED1" library="Master 2016" deviceset="LED" device="1206"/>
-<part name="JP3" library="SparkFun-Passives" deviceset="JUMPER-2" device="PTH" value="Signals"/>
+<part name="JP3" library="SparkFun-Passives" deviceset="JUMPER-2" device="PTH" value="LED En"/>
 <part name="C2" library="Master 2016" deviceset="CPOL-EU" device="E2.5-5**10UF" value="1u"/>
 <part name="GND13" library="Master" deviceset="GND" device=""/>
@@
 <part name="GND10" library="Master" deviceset="GND" device=""/>
 <part name="GND12" library="Master" deviceset="GND" device=""/>
-<part name="J1" library="SparkFun-Connectors" deviceset="CONN_03" device="" value="455-1750-1-ND"/>
+<part name="J1" library="SparkFun-Connectors" deviceset="CONN_03" device="" value="Thermo Rly"/>
 <part name="LED3" library="Master 2016" deviceset="LED" device="1206"/>
 <part name="LED4" library="Master 2016" deviceset="LED" device="1206"/>
@@
 <part name="P1" library="con-jst-eh" deviceset="B5B-EH-A" device="" value="X10A"/>
 <part name="J2" library="conn-jst-pa6" deviceset="B06B-PASK(LF)(SN)" device="" value="X85A - PL"/>
+<part name="JP5" library="SparkFun-Passives" deviceset="JUMPER-2" device="PTH" value="SG En"/>
 </parts>
 <sheets>
@@
 <attribute name="VALUE" x="78.4606" y="67.5386" size="2.0828" layer="96" ratio="6" rot="SR0"/>
 </instance>
+<instance part="JP5" gate="A" x="-35.56" y="45.72" smashed="yes">
+<attribute name="NAME" x="-36.83" y="45.72" size="1.778" layer="95" rot="R90"/>
+<attribute name="VALUE" x="-29.845" y="45.72" size="1.778" layer="96" rot="R90"/>
+</instance>
 </instances>
 <busses>
@@
 </segment>
 <segment>
-<pinref part="K1" gate="A" pin="2"/>
-<wire x1="-76.2" y1="35.56" x2="-76.2" y2="40.64" width="0.1524" layer="91"/>
-<label x="-76.2" y="40.64" size="1.27" layer="95" rot="R90" xref="yes"/>
-</segment>
-<segment>
-<pinref part="K2" gate="A" pin="2"/>
-<wire x1="-45.72" y1="35.56" x2="-45.72" y2="43.18" width="0.1524" layer="91"/>
-<label x="-45.72" y="43.18" size="1.27" layer="95" rot="R90" xref="yes"/>
+<label x="-22.86" y="43.18" size="1.27" layer="95" xref="yes"/>
+<pinref part="JP5" gate="A" pin="2"/>
+<wire x1="-22.86" y1="43.18" x2="-33.02" y2="43.18" width="0.1524" layer="91"/>
 </segment>
 <segment>
@@
 </segment>
 </net>
+<net name="N$6" class="0">
+<segment>
+<pinref part="K1" gate="A" pin="2"/>
+<wire x1="-76.2" y1="35.56" x2="-76.2" y2="43.18" width="0.1524" layer="91"/>
+<wire x1="-76.2" y1="43.18" x2="-45.72" y2="43.18" width="0.1524" layer="91"/>
+<pinref part="K2" gate="A" pin="2"/>
+<wire x1="-45.72" y1="43.18" x2="-45.72" y2="35.56" width="0.1524" layer="91"/>
+<pinref part="JP5" gate="A" pin="1"/>
+<wire x1="-45.72" y1="43.18" x2="-35.56" y2="43.18" width="0.1524" layer="91"/>
+<junction x="-45.72" y="43.18"/>
+</segment>
+</net>

Commit message: I think this is v1.0. This commit free of any panelisation guff.
Parts:
- removed SG: (no value), SparkFun-Connectors:CONN_04LOCK
- added CONN4: SG, SparkFun-Connectors:CONN_04PTH
- added LED5: (no value), Master 2016:LED1206
- added R17: 180R, Master 2016:R-EU_
- U1: value TLP291-4(GB-TP,E) -> TLP291-4
- U2: value AP2112K-3.3TRG1 -> AP2112K-3.3
- renumbered J1 to CON5, J2 to CON2, P1 to CON3, R19 to R16, SJ3 to SJ1, SV1 to CON1
Connections:
- new net N$28: LED5.C, R17.2
- net GPIO2: now also R17.1
- net N$22: now also CONN4.1; no longer SG.1
- net N$23: now also CONN4.2; no longer SG.2
- net N$24: now also CONN4.3; no longer SG.3
- net N$25: now also CONN4.4; no longer SG.4
- net VCC: now also LED5.A
Other:
- note added: "Device substitution: for RTS Reset, 1N5711, use BAT48"
- note added: "Pins 2-5 pulled high by heat pump when transistors are off. Separate ground shown but actually X85A GND is same as X10A GND."
- note added: "R17, LED5 optional (gpio2 typically drives LED on ESP12)"
- note added: "SG and Power Limitation share GPIOs, so ONLY ONE may be used"
- note removed: "Device substitutions: for LDO, AP2112K-3.3, use MIC5504-3.3 for RTS Reset, 1N5711, use BAT48"
- moved on the sheet: LED1, LED2, LED3, LED4, R12, R13, R14, R15, R5
